Commit message: more compatibility changes

File: src/husky_ur3_bringup/urdf/accessories/d435_camera_g.urdf.xacro (robot description, xacro)
@@ -1,7 +1,17 @@
 <?xml version="1.0"?>
+<!-- File: g_sensor_d435.urdf.xacro
+     Purpose: Define a D435-like depth camera link with a COMPLETE inertial,
+     so robot_state_publisher/URDF parser doesn’t error on missing ixy, etc. -->
 <robot name="g_sensor_d435" xmlns:xacro="http://ros.org/wiki/xacro">
+  <!--
+    Macro params:
+      parent: parent link to mount the camera to
+      *origin: xacro block with <origin .../> passed at callsite
+      name: base name for links/joints; default "g_camera" => g_camera_link, g_camera_joint
+      use_nominal_extrinsics: unused here, kept for compatibility
+  -->
   <xacro:macro name="g_sensor_d435" params="parent *origin name:=g_camera use_nominal_extrinsics:=true">
     <xacro:property name="M_PI" value="3.1415926535897931" />
-    <!-- Fixed mounting joint -->
+    <!-- Fixed mount to the parent -->
     <joint name="${name}_joint" type="fixed">
       <xacro:insert_block name="origin" />
@@ -9,5 +19,5 @@
       <child link="${name}_link" />
     </joint>
-    <!-- Physical camera body -->
+    <!-- Physical camera body (visual + collision + COMPLETE inertial) -->
     <link name="${name}_link">
       <visual>
@@ -26,11 +36,13 @@
         </geometry>
       </collision>
+      <!-- IMPORTANT: all six inertia terms are present -->
       <inertial>
-        <mass value="0.072"/>
+        <mass value="0.1"/>
         <origin xyz="0 0 0"/>
-        <inertia ixx="0.0039" iyy="0.0005" izz="0.0039"/>
+        <inertia ixx="0.001" ixy="0.0" ixz="0.0"
+                 iyy="0.001" iyz="0.0" izz="0.001"/>
       </inertial>
     </link>
-    <!-- Gazebo Sim sensor -->
+    <!-- Gazebo Sim depth camera sensor (topic name is arbitrary) -->
     <gazebo reference="${name}_link">
       <sensor name="${name}_sensor" type="depth_camera">

Commit message: Decent midway

File: src/husky_ur3_bringup/urdf/accessories/d435_camera_g.urdf.xacro (robot description, xacro)
@@ -46,5 +46,5 @@
     <!-- Gazebo Sim depth camera sensor (topic name is arbitrary) -->
     <gazebo reference="${name}_link">
-      <sensor name="${name}_sensor" type="depth_camera">
+      <sensor name="${name}_sensor" type="rgbd_camera">
         <always_on>true</always_on>
         <update_rate>20.0</update_rate>

File: src/husky_ur3_bringup/urdf/accessories/d435_camera_h.urdf.xacro (robot description, xacro)
@@ -34,5 +34,5 @@
     <!-- Gazebo Sim native depth camera (RGB‑D replacement) -->
     <gazebo reference="${name}_link">
-      <sensor name="${name}_depth_camera" type="depth_camera">
+      <sensor name="${name}_depth_camera" type="rgbd_camera">
         <always_on>true</always_on>
         <update_rate>20.0</update_rate>

File: src/husky_ur3_bringup/urdf/accessories/sick_tim571.urdf.xacro (robot description, xacro)
@@ -35,5 +35,5 @@
     <xacro:sensor_sick_tim571_gazebo/>
   </xacro:macro>
-  <xacro:macro name="sensor_sick_tim571_gazebo">
+  <!-- <xacro:macro name="sensor_sick_tim571_gazebo">
     <gazebo reference="${prefix}_link">
       <sensor name="${prefix}_lidar" type="gpu_lidar">
@@ -66,4 +66,29 @@
       </sensor>
     </gazebo>
+  </xacro:macro> -->
+  <xacro:macro name="sensor_sick_tim571_gazebo">
+    <gazebo reference="${prefix}_link">
+      <sensor name="${prefix}_lidar" type="gpu_lidar">
+        <topic>/scan</topic>
+        <update_rate>15</update_rate>
+        <gz_frame_id>${prefix}_link</gz_frame_id>
+        <lidar>
+          <scan>
+            <horizontal>
+              <samples>716</samples>
+              <resolution>1</resolution>
+              <min_angle>${min_angle}</min_angle>
+              <max_angle>${max_angle}</max_angle>
+            </horizontal>
+          </scan>
+          <range>
+            <min>0.05</min>
+            <max>25.0</max>
+            <resolution>0.01</resolution>
+          </range>
+        </lidar>
+        <visualize>true</visualize>
+      </sensor>
+    </gazebo>
   </xacro:macro>
 </robot>

File: src/husky_ur3_bringup/urdf/husky_ur3_gripper.urdf.xacro (robot description, xacro)
@@ -165,4 +165,37 @@
    	<origin xyz="$(arg laser_xyz)" rpy="$(arg laser_rpy)"/>
   </xacro:sensor_sick_tim571>
+  <!-- Simple Gazebo Sim lidar sensor on top_plate_link -->
+  <!-- <link name="lidar_link">
+    <inertial>
+      <mass value="0.1"/>
+      <origin xyz="0 0 0"/>
+      <inertia ixx="1e-4" ixy="0" ixz="0" iyy="1e-4" iyz="0" izz="1e-4"/>
+    </inertial>
+  </link>
+  <joint name="lidar_joint" type="fixed">
+    <parent link="top_plate_link"/>
+    <child link="lidar_link"/>
+    <origin xyz="0.3 0.0 0.2" rpy="0 0 0"/>
+  </joint>
+  <gazebo reference="lidar_link">
+    <sensor name="lidar" type="lidar">
+      <pose>0 0 0 0 0 0</pose>
+      <update_rate>10</update_rate>
+      <topic>/lidar</topic>
+      <lidar>
+        <horizontal>
+          <samples>720</samples>
+          <resolution>1</resolution>
+          <min_angle>-1.57</min_angle>
+          <max_angle> 1.57</max_angle>
+        </horizontal>
+        <range>
+          <min>0.1</min>
+          <max>30.0</max>
+          <resolution>0.01</resolution>
+        </range>
+      </lidar>
+    </sensor>
+  </gazebo> -->
  <joint name="control_box_ur3_joint" type="fixed">
       <origin xyz="-0.095 0 0.233" rpy="${M_PI/2} 0 0" />
@@ -211,4 +244,9 @@
     </plugin>
   </gazebo>
+<gazebo>
+  <plugin filename="gz-sim-sensors-system" name="gz::sim::systems::Sensors">
+    <render_engine>ogre2</render_engine>
+  </plugin>
+</gazebo>
 <!--
   <gazebo>
